Commit message: add go2w model

File: robots/yuelu_description/urdf/yuelu_description.urdf (robot description, URDF)
Before this commit: robot yuelu, 7 links, 6 joints
Links:
- link base_link: geometry collision mesh filename=package://yuelu_description/meshes/base_link.STL; visual mesh filename=package://yuelu_description/meshes/base_link.STL
- link l_wheel_Link: geometry collision cylinder length=0.022 radius=0.078; visual mesh filename=package://yuelu_description/meshes/l_wheel_Link.STL
- link lf0_Link: geometry collision mesh filename=package://yuelu_description/meshes/lf0_Link.STL; visual mesh filename=package://yuelu_description/meshes/lf0_Link.STL
- link lf1_Link: geometry collision mesh filename=package://yuelu_description/meshes/lf1_Link.STL; visual mesh filename=package://yuelu_description/meshes/lf1_Link.STL
- link r_wheel_Link: geometry collision cylinder length=0.022 radius=0.078; visual mesh filename=package://yuelu_description/meshes/r_wheel_Link.STL
- link rf0_Link: geometry collision mesh filename=package://yuelu_description/meshes/rf0_Link.STL; visual mesh filename=package://yuelu_description/meshes/rf0_Link.STL
- link rf1_Link: geometry collision mesh filename=package://yuelu_description/meshes/rf1_Link.STL; visual mesh filename=package://yuelu_description/meshes/rf1_Link.STL
